File: circuit/logger_v2/logger_v2.kicad_pcb (KiCad board)
At the start: 4 copper layers, 68.7 x 53.4 mm, 98 parts, among them J1 Power, J10 S-037-TGG, J11 2452796-1, J12 47219-2001, J2 Analog, J3 Digital/PWM, J4 Digital/PWM, J5 Conn_01x02_Pin, J6 43045-0400, J7 S-037-TGG, J8 Conn_01x02_Pin, J9 43045-0400, Q1 2N7002, U1 BNO055_module, U10 USBLC6-4SC6, U2 AP63301WU-7, U3 TXU0204PWR, U4 MCP25625-E/SS, U5 MAX-M10M-00B, U6 SIM7070G, U7 ATA6561-GAQW, U8 TC74HC595AF, U9 USBLC6-4SC6, Y1 20MHz CL10pF

Commit message: Save current logger, UPS, firmware, and verification artifacts
Parts:
- moved R15 0.96 mm to (74.6, 92.7)
- moved J7 0.57 mm to (74.5, 86.5)
- moved J10 0.27 mm to (74.5, 77.0)
Routing:
- net +3V3: track 102.1 -> 103.8 mm
- net /IMU_INT: track 57.2 -> 58.9 mm
- net Net-(D2-A2): track 9.05 -> 10.1 mm
- net /~{IMU_RESET}: track 45.2 -> 45.7 mm
- net GND: vias 272 -> 279
