File: circuit/logger_v2/logger_v2.kicad_sch (KiCad schematic)
At the start: 98 parts, among them J1 Power, J10 S-037-TGG, J11 2452796-1, J12 47219-2001, J2 Analog, J3 Digital/PWM, J4 Digital/PWM, J5 Conn_01x02_Pin, J6 43045-0400, J7 S-037-TGG, J8 Conn_01x02_Pin, J9 43045-0400, Q1 2N7002, U1 BNO055_module, U10 USBLC6-4SC6, U2 AP63301WU-7, U3 TXU0204PWR, U4 MCP25625-E/SS, U5 MAX-M10M-00B, U6 SIM7070G, U7 ATA6561-GAQW, U8 TC74HC595AF, U9 USBLC6-4SC6, Y1 20MHz CL10pF

Commit message: Save current logger, UPS, firmware, and verification artifacts
Parts:
- C1, C12, C13, C2, C28, C8: JLCPCB_Class Basic -> (none); LCSC C15850 -> (none); MPN GRM21BR71A106KE51 -> CL21B106KPQNFNE; Manufacturer Samsung -> Samsung Electro-Mechanics; SelectionNote (none) -> 旧445-6857-1-NDが注文画面で入荷待ちのため差替え。Samsung製10µF±10%・10V・X7R、2.0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; Specification 10uF X5R 25V 0805 -> 10µF ±10% X7R 10V; 0805 / 2012; Supplier 秋月電子通商 -> DigiKey; SupplierCode 117593 -> 1276-2934-1-ND; SupplierURL https://akizukidenshi.com/catalog/g/g117593/ -> https://www.digikey.jp/en/products/detail/samsung-electro-m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
- C10, C9: JLCPCB_Class Basic -> (none); LCSC C1647 -> (none); MPN CC0603N150J500 -> CC0603JRNPO9BN150; Manufacturer Samsung -> Yageo; SelectionNote (none) -> Value=15pを採用。古いSpecificationの18pF/CL12pFは不採用。 少量価格の段差も考慮して1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; Specification 18pF C0G 50V 5%; 20MHz CL12pF crystal -> 15pF ±5% C0G 50V; 0603 / 1608; Supplier 秋月電子通商 -> DigiKey; SupplierCode 113312 -> 311-1060-1-ND; SupplierURL https://akizukidenshi.com/catalog/g/g113312/ -> https://www.digikey.jp/en/products/detail/yageo/CC0603JRNPO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
- C11: JLCPCB_Class Basic -> (none); LCSC C14663 -> (none); MPN GRM188B11H103KA01 -> GRM188R72A103KA01D; Manufacturer Yageo -> Murata Electronics; SelectionNote RF給電バイパス。B特性、-25～85℃ -> 現行Value=0.01u。耐圧は元の50V以上。 少量価格の段差も考慮して10個。; Specification 100nF X7R 50V 0603 -> 10nF ±10% X7R 100V; 0603 / 1608; Supplier 秋月電子通商 -> DigiKey; SupplierCode 113387 -> 490-GRM188R72A103KA01DCT-ND; SupplierURL https://akizukidenshi.com/catalog/g/g113387/ -> https://www.digikey.jp/en/products/detail/murata-electronic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
- C14, C17, C19, C21, C22, C23, C24, C25, C26, C27, C3, C4, C5, C6: JLCPCB_Class Basic -> (none); LCSC C14663 -> (none); Manufacturer Yageo -> Murata Electronics; SelectionNote (none) -> 現行MPNを維持。C21～C27も現行Value=0.1u。; Specification 100nF X7R 50V 0603 -> 100nF ±10% X7R 100V; 0603 / 1608; Supplier 秋月電子通商 -> DigiKey; SupplierCode 114559 -> 490-3285-1-ND; SupplierURL https://akizukidenshi.com/catalog/g/g114559/ -> https://www.digikey.jp/en/products/detail/murata-electronic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
- C15: MPN C2012X7R1H105KT000N -> C2012X7R1H105K085AC; SelectionNote Same footprint as V1 1uF. V1 does not specify an exact MPN. -> 同サイズ・同容量・同耐圧。高さ最大1.0mm。新規設計非推奨品だが在庫表示あり。; Specification 1uF 50V X7R, 0805 (2012 metric) -> 1µF ±10% X7R 50V; 0805 / 2012; Supplier 秋月電子通商 -> DigiKey; SupplierCode 115331 -> 445-14539-1-ND; SupplierURL https://akizukidenshi.com/catalog/g/g115331/ -> https://www.digikey.jp/en/products/detail/tdk-corporation/C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
- C20: MPN C2012X7R1H105KT000N -> CL21B106KPQNFNE; Manufacturer TDK -> Samsung Electro-Mechanics; SelectionNote Same footprint as V1 1uF. V1 does not specify an exact MPN. -> 旧445-6857-1-NDが注文画面で入荷待ちのため差替え。Samsung製10µF±10%・10V・X7R、2.0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; Specification 1uF 50V X7R, 0805 (2012 metric) -> 10µF ±10% X7R 10V; 0805 / 2012; Supplier 秋月電子通商 -> DigiKey; SupplierCode 115331 -> 1276-2934-1-ND; SupplierURL https://akizukidenshi.com/catalog/g/g115331/ -> https://www.digikey.jp/en/products/detail/samsung-electro-m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
- C7: Manufacturer Panasonic -> Panasonic Industry; SelectionNote OS-CON SVPC; pad 1 positive +3V8, pad 2 negative GND. Gener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 -> 指定品維持。ESR17mΩ、極性あり。; Specification 330uF 6.3V conductive polymer aluminum, ESR 17mOhm, D6.3 x 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 -> 330µF 6.3V ポリマー; φ6.3 × H5.9mm; SupplierURL https://www.digikey.jp/ja/products/detail/panasonic-industr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 -> https://www.digikey.jp/en/products/detail/panasonic-industr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
- D1, D4: JLCPCB_Class Extended -> (none); LCSC C14486 -> (none); MPN PEC3824C2A-AU_R1_000A1 -> ESDCAN24-2BLY; Manufacturer onsemi -> STMicroelectronics; SelectionNote CAN用24V双方向TVS、1/2=bus、3=GND -> PEC3824C2A-AUの代替。1/2=CAN、3=GND。24V、Vbr最低27V、容量最大30pF。クランプ特性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; Specification (none) -> CAN用 双方向2線 TVS 24V; SOT-23-3; Supplier 秋月電子通商 -> DigiKey; SupplierCode 129497 -> 497-13262-1-ND; SupplierURL https://akizukidenshi.com/catalog/g/g129497/ -> https://www.digikey.jp/en/products/detail/stmicroelectronic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
- D10, D11, D12, D5, D6, D7, D8, D9: JLCPCB_Class Basic -> (none); LCSC C2297 -> (none); MPN OSG80805C1C -> LTST-C170KGKT; Manufacturer Hubei KENTO Elec -> Lite-On; SelectionNote 黄緑570nm、2012、VF typ 2V -> 同0805、1=カソード、2=アノード。元品と発光色・明るさに差あり。; Specification (none) -> 緑LED 571nm / Vf約2V; 0805 / 2012; Supplier 秋月電子通商 -> DigiKey; SupplierCode 106421 -> 160-1414-1-ND; SupplierURL https://akizukidenshi.com/catalog/g/g106421/ -> https://www.digikey.jp/en/products/detail/liteon/LTST-C170K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
- D2: JLCPCB_Class Extended -> (none); LCSC C45961 -> (none); MPN PESD5V0F1BL-Q -> AQ3045-01ETG; Manufacturer Nexperia -> Littelfuse; SelectionNote RF用双方向TVS、VRWM5.5V、Ctyp0.4pF / max0.55pF -> GNSSアンテナESD用の機能代替。SOD882・端子ピッチ0.65mm、現PCBの0.4×0.7mmパッドに端子が重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; Specification (none) -> RF用 双方向TVS 5.3V / 0.35pF; SOD882 / 1.0×0.6mm; Supplier 他社調達 -> DigiKey; SupplierCode (none) -> F9321CT-ND; SupplierURL https://www.nexperia.com/product/PESD5V0F1BL-Q -> https://www.digikey.jp/en/products/detail/littelfuse-inc/AQ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
- D3: MPN (none) -> CSPSBHC4V5LB-TP; Manufacturer (none) -> MCC; SelectionNote (none) -> 3.8V電源ESD用の機能代替。4.5V双方向、端子ピッチ0.65mm・長さ0.20～0.30/幅0.45～0.55m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; Specification (none) -> LTE電源 双方向TVS 4.5V; CSP1006-2 / 1.0×0.6mm; Supplier (none) -> DigiKey; SupplierCode (none) -> 353-CSPSBHC4V5LB-TPCT-ND; SupplierURL (none) -> https://www.digikey.jp/en/products/detail/mcc-micro-commerc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
- J11: Manufacturer (none) -> TE Connectivity; SelectionNote ユーザー指定RS 286-8822、維持 -> SDとは別部品。現行指定品維持。マーケットプレイス品ではなくDigiKey直販CTを指定。; Specification (none) -> nanoSIM ヒンジ式ソケット; TE専用フットプリント; Supplier 他社調達 -> DigiKey; SupplierCode (none) -> 343-2452796-1CT-ND; SupplierURL https://jp.rs-online.com/web/p/memory-card-connectors/28688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 -> https://www.digikey.jp/en/products/detail/te-connectivity-l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
- J6, J9: Manufacturer (none) -> Molex; SelectionNote 既存ケーブルとの嵌合を維持する例外 -> 43045-0400と同じ品番の表記違い。指定どおり2個だけ。ケーブル側・圧着端子は含めない。; Specification (none) -> Micro-Fit 3.0 基板側4極; 2×2 / 3.0mm 横向きTHT; Supplier 他社調達 -> DigiKey; SupplierCode (none) -> WM1814-ND; SupplierURL https://www.molex.com/en-us/products/part-detail/430450400 -> https://www.digikey.jp/en/products/detail/molex/0430450400/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
- L1: MPN DFE252012P-2R2M=P2 -> DFE252012F-2R2M=P2; Manufacturer Murata -> Murata Electronics; SelectionNote User selected 2520. Verify temperature and startup/overload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 -> 旧490-10649-1-NDがユーザーのカートで規制表示のためFシリーズへ差替え。2.2µH±20%、外形・高さ・推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; Specification 2.2uH +/-20%, 2.2A temperature-rise current, 3.0A at 30% L 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 -> 2.2µH ±20% 電源インダクタ; 2.5×2.0×1.2mm; SupplierCode 490-10649-1-ND -> 490-13055-1-ND; SupplierURL https://www.digikey.com/en/products/detail/murata-electroni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 -> https://www.digikey.jp/en/products/detail/murata-electronic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
- L2: Manufacturer Murata -> Murata Electronics; SelectionNote Same MPN and nominal footprint as LoggerV1 L1. -> 指定品維持。440mA、SRF3.7GHz以上。一般電源用インダクタには置換しない。; Specification 27nH RF wirewound, 440mA, DCR 0.21ohm max, SRF 3.7GHz min -> 27nH RF巻線インダクタ; 0603 / 1608; SupplierCode (none) -> 490-1174-1-ND; SupplierURL https://www.digikey.jp/ja/products/detail/murata-electronic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 -> https://www.digikey.jp/en/products/detail/murata-electronic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
- Q1: MPN 2N7002 -> 2N7002ET1G; Manufacturer (none) -> onsemi; SelectionNote (none) -> 2N7002相当。1=G、2=S、3=Dで基板と一致。; Specification (none) -> Nch MOSFET 60V; SOT-23; Supplier 秋月電子通商 -> DigiKey; SupplierCode 103919 -> 2N7002ET1GOSCT-ND; SupplierURL https://akizukidenshi.com/catalog/g/g103919/ -> https://www.digikey.jp/en/products/detail/onsemi/2N7002ET1G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
- R1, R11, R5: JLCPCB_Class Basic -> (none); LCSC C25804 -> (none); MPN RK73B1JTTD103J -> CRT0603-BY-1003ELF; Manufacturer UNI-ROYAL -> Bourns; SelectionNote (none) -> 0603・100kΩ・0.1%・0.1W。R11の帰還精度を優先し同一品へ統一。; Specification (none) -> 100kΩ ±0.1% 0.1W; 0603 / 1608; Supplier 秋月電子通商 -> DigiKey; SupplierCode 130355 -> CRT0603-BY-1003ELFCT-ND; SupplierURL https://akizukidenshi.com/catalog/g/g130355/ -> https://www.digikey.jp/en/products/detail/bourns-inc/CRT060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
- R10: JLCPCB_Class Basic -> (none); LCSC C25804 -> (none); MPN RK73B1JTTD103J -> RC0603FR-07374KL; Manufacturer UNI-ROYAL -> Yageo; SelectionNote (none) -> 電源帰還上側。Value=374kを採用。 少量価格の段差も考慮して10個。; Specification (none) -> 374kΩ ±1% 0.1W; 0603 / 1608; Supplier 秋月電子通商 -> DigiKey; SupplierCode 130355 -> 311-374KHRCT-ND; SupplierURL https://akizukidenshi.com/catalog/g/g130355/ -> https://www.digikey.jp/en/products/detail/yageo/RC0603FR-07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
- R14, R16: JLCPCB_Class Basic -> (none); LCSC C22787 -> (none); MPN RC0603J120R -> RC0603FR-07120RL; Manufacturer UNI-ROYAL -> Yageo; SelectionNote リール販売。CAN終端定格は別途確認、現在の1608を維持 -> 現行DNP=noのため含む。接続するCANバスの終端配置に従って実装する。 少量価格の段差も考慮して10個。; Specification (none) -> 120Ω ±1% 0.1W; 0603 / 1608; Supplier 秋月電子通商 -> DigiKey; SupplierCode 130332 -> 311-120HRCT-ND; SupplierURL https://akizukidenshi.com/catalog/g/g130332/ -> https://www.digikey.jp/en/products/detail/yageo/RC0603FR-07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
- R15: JLCPCB_Class Extended -> (none); LCSC C25478 -> (none); MPN CRCW251227R0JNEG -> RMCF2512JT27R0; Manufacturer UNI-ROYAL -> Stackpole Electronics; SelectionNote 27Ω 5% 1W、短絡時最悪約0.468W。基板温度・放熱を確認 -> 2512・27Ω・5%・1Wを維持。同サイズのStackpole品へ置換。; Specification 27ohm 5% 1W; verify antenna supply under load -> 27Ω ±5% 1W; 2512 / 6332; Supplier 他社調達 -> DigiKey; SupplierCode (none) -> RMCF2512JT27R0CT-ND; SupplierURL https://www.vishay.com/docs/20035/dcrcwe3.pdf -> https://www.digikey.jp/en/products/detail/stackpole-electro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
- R17, R18, R19: JLCPCB_Class Basic -> (none); LCSC C25804 -> (none); MPN RK73B1JTTD103J -> CRCW060322R0FKEA; Manufacturer UNI-ROYAL -> Vishay Dale; SelectionNote (none) -> 0603・22Ω・1%・0.1Wを維持。在庫表示のあるVishay品。; Specification (none) -> 22Ω ±1% 0.1W; 0603 / 1608; Supplier 秋月電子通商 -> DigiKey; SupplierCode 130355 -> 541-22.0HCT-ND; SupplierURL https://akizukidenshi.com/catalog/g/g130355/ -> https://www.digikey.jp/en/products/detail/vishay-dale/CRCW0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
- R20, R21: JLCPCB_Class Basic -> (none); LCSC C25804 -> (none); MPN RK73B1JTTD103J -> RC0603JR-070RL; Manufacturer UNI-ROYAL -> Yageo; SelectionNote (none) -> 現行Value=0Ω。 少量価格の段差も考慮して10個。; Specification (none) -> 0Ω ジャンパ 0.1W; 0603 / 1608; Supplier 秋月電子通商 -> DigiKey; SupplierCode 130355 -> 311-0.0GRCT-ND; SupplierURL https://akizukidenshi.com/catalog/g/g130355/ -> https://www.digikey.jp/en/products/detail/yageo/RC0603JR-07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
- R22, R6, R8: JLCPCB_Class Basic -> (none); LCSC C25819 -> (none); MPN RC0603J47K -> RC0603FR-0747KL; Manufacturer UNI-ROYAL -> Yageo; SelectionNote リール販売 -> 同サイズの1%品。; Specification (none) -> 47kΩ ±1% 0.1W; 0603 / 1608; Supplier 秋月電子通商 -> DigiKey; SupplierCode 129458 -> 311-47.0KHRCT-ND; SupplierURL https://akizukidenshi.com/catalog/g/g129458/ -> https://www.digikey.jp/en/products/detail/yageo/RC0603FR-07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
- R23, R24, R25, R26, R27, R28, R29, R30: JLCPCB_Class Basic -> (none); LCSC C23228 -> (none); MPN RK73B1JTTD102J -> RC0603FR-071KL; Manufacturer UNI-ROYAL -> Yageo; SelectionNote LED電流 約1.3mA @3.3V、VF=2V -> Value基準。古いMPNに10kΩ表記が残る箇所あり。; Specification (none) -> 1kΩ ±1% 0.1W; 0603 / 1608; Supplier 秋月電子通商 -> DigiKey; SupplierCode 130351 -> 311-1.00KHRCT-ND; SupplierURL https://akizukidenshi.com/catalog/g/g130351/ -> https://www.digikey.jp/en/products/detail/yageo/RC0603FR-07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
- R31, R32: JLCPCB_Class Basic -> (none); LCSC C25804 -> (none); MPN RK73B1JTTD103J -> RC0603FR-0747KL; Manufacturer UNI-ROYAL -> Yageo; SelectionNote (none) -> 同サイズの1%品。; Specification (none) -> 47kΩ ±1% 0.1W; 0603 / 1608; Supplier 秋月電子通商 -> DigiKey; SupplierCode 130355 -> 311-47.0KHRCT-ND; SupplierURL https://akizukidenshi.com/catalog/g/g130355/ -> https://www.digikey.jp/en/products/detail/yageo/RC0603FR-07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
- R4: JLCPCB_Class Basic -> (none); LCSC C25804 -> (none); MPN RK73B1JTTD103J -> RC0603FR-071KL; Manufacturer UNI-ROYAL -> Yageo; SelectionNote (none) -> Value基準。古いMPNに10kΩ表記が残る箇所あり。; Specification (none) -> 1kΩ ±1% 0.1W; 0603 / 1608; Supplier 秋月電子通商 -> DigiKey; SupplierCode 130355 -> 311-1.00KHRCT-ND; SupplierURL https://akizukidenshi.com/catalog/g/g130355/ -> https://www.digikey.jp/en/products/detail/yageo/RC0603FR-07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
- U10, U9: MPN USBLC6-4SC6 -> USBLC6-4SC6Y; Manufacturer (none) -> STMicroelectronics; SelectionNote SIM/SD用低容量ESD。秋月適合品未確認、維持 -> USBLC6-4SC6の車載グレード品。同じ4線・SOT23-6・ピン配置。2=GND、5=VBUS、1/3/4/6=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; Specification (none) -> 4線ESD保護; SOT-23-6; Supplier 他社調達 -> DigiKey; SupplierCode (none) -> 497-11883-1-ND; SupplierURL https://www.st.com/en/protection-devices/usblc6-4.html -> https://www.digikey.jp/en/products/detail/stmicroelectronic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
- U2: Manufacturer (none) -> Diodes Incorporated; SelectionNote 0.95mm pitch, no exposed pad; DigiKey stock confirmed 2026-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 -> 指定品維持。AP63300/固定電圧版と混同しない。; Specification (none) -> 3A 降圧DC/DC; TSOT26; SupplierURL https://www.digikey.jp/ja/products/detail/diodes-incorporat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 -> https://www.digikey.jp/en/products/detail/diodes-incorporat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
- U3: Manufacturer (none) -> Texas Instruments; SelectionNote 2Mbps UART 1.8/3.3V変換用。旧案の2個目は購入数量から除く -> 指定品維持。PWパッケージ。; Specification (none) -> 4bit レベル変換; TSSOP-14 / P0.65; Supplier 他社調達 -> DigiKey; SupplierCode (none) -> 296-TXU0204PWRCT-ND; SupplierURL https://www.ti.com/product/TXU0204 -> https://www.digikey.jp/en/products/detail/texas-instruments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
- U4: JLCPCB_Class Extended -> (none); LCSC C184944 -> (none); Manufacturer Microchip -> Microchip Technology; SelectionNote (none) -> 指定品維持。/SSパッケージ。高価なため予備なし。; Specification (none) -> CANコントローラ＋トランシーバ; SSOP-28 / 幅5.3mm; Supplier 秋月電子通商 -> DigiKey; SupplierCode 112663 -> MCP25625T-E/SSCT-ND; SupplierURL https://akizukidenshi.com/catalog/g/g112663/ -> https://www.digikey.jp/en/products/detail/microchip-technol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
- U6: Manufacturer (none) -> SIMCom; SelectionNote 指定部品、秋月制約の対象外 -> 指定の裸モジュール。開発ボードではない。高価なため予備なし。; Specification (none) -> LTE Cat-M/NB-IoTモジュール; LCC-68 / 24×24mm; Supplier 他社調達 -> DigiKey; SupplierCode (none) -> 3781-SIM7070G-ND; SupplierURL https://en.simcom.com/product/SIM7070G.html -> https://www.digikey.jp/en/products/detail/simcom-wireless-s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
- U7: JLCPCB_Class Extended -> (none); LCSC C2929602 -> (none); Manufacturer Microchip -> Microchip Technology; SelectionNote (none) -> 指定品維持。VDFN版を選ばない。; Specification (none) -> CANトランシーバ; SOIC-8 / 幅3.9mm; Supplier 秋月電子通商 -> DigiKey; SupplierCode 130008 -> ATA6561-GAQW-NCT-ND; SupplierURL https://akizukidenshi.com/catalog/g/g130008/ -> https://www.digikey.jp/en/products/detail/microchip-technol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
- U8: JLCPCB_Class Basic -> (none); LCSC C5947 -> (none); MPN TC74HC595AF -> TC74HC595AF(EL,F); Manufacturer Nexperia -> Toshiba; SelectionNote (none) -> 指定AFのSOP16を維持。一般的な幅3.9mm SOICの74HC595は合わない。; Specification (none) -> 8bit シフトレジスタ; SOP-16 / 幅5.3mm; Supplier 秋月電子通商 -> DigiKey; SupplierCode 110077 -> 264-TC74HC595AF(EL,F)CT-ND; SupplierURL https://akizukidenshi.com/catalog/g/g110077/ -> https://www.digikey.jp/en/products/detail/toshiba-semicondu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
- Y1: JLCPCB_Class Extended -> (none); LCSC C18213008 -> (none); MPN 20M10PB/XT324-10/80 -> ABM8-20.000MHZ-10-B1U-T; Manufacturer YXC -> Abracon; SelectionNote C2/C3=15pF; stray 2.5pF仮定、発振余裕と周波数を実機確認 -> 同寸法3.2×2.5mm、CL10pF。1/3=水晶、2/4=GND。発振余裕は実機で確認。; Specification (none) -> 水晶 20MHz / CL10pF; 3225 / 4端子; Supplier 秋月電子通商 -> DigiKey; SupplierCode 130244 -> 535-14973-1-ND; SupplierURL https://akizukidenshi.com/catalog/g/g130244/ -> https://www.digikey.jp/en/products/detail/abracon-llc/ABM8-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
